Commit message: Quadruped

File: body.urdf (robot description, URDF)
Before this commit: robot robot, 3 links, 2 joints
Links:
- added link Backarm, mass 1; collision box size=0.19999999999999996 0.19999999999999996 1; visual box size=0.19999999999999996 0.19999999999999996 1
- added link Frontarm, mass 1; collision box size=0.19999999999999996 0.19999999999999996 1; visual box size=0.19999999999999996 0.19999999999999996 1
- added link Leftarm, mass 1; collision box size=0.19999999999999996 0.19999999999999996 1; visual box size=0.19999999999999996 0.19999999999999996 1
- added link Leftleg, mass 1; collision box size=1 0.19999999999999996 0.19999999999999996; visual box size=1 0.19999999999999996 0.19999999999999996
- added link Rightarm, mass 1; collision box size=0.19999999999999996 0.19999999999999996 1; visual box size=0.19999999999999996 0.19999999999999996 1
- added link Rightleg, mass 1; collision box size=1 0.19999999999999996 0.19999999999999996; visual box size=1 0.19999999999999996 0.19999999999999996
- link Backleg: geometry collision box size=0.19999999999999996 1 0.19999999999999996; visual box size=0.19999999999999996 1 0.19999999999999996
- link Frontleg: geometry collision box size=0.19999999999999996 1 0.19999999999999996; visual box size=0.19999999999999996 1 0.19999999999999996
Joints:
- added joint Backleg_Backarm: type revolute, parent Backleg, child Backarm, origin xyz=0 -1 0 rpy=0 0 0, axis 1 0 0, limit lower=-3.14159 upper=3.14159 effort=0.0 velocity=0.0
- added joint Frontleg_Frontarm: type revolute, parent Frontleg, child Frontarm, origin xyz=0 1 0 rpy=0 0 0, axis 1 0 0, limit lower=-3.14159 upper=3.14159 effort=0.0 velocity=0.0
- added joint Leftleg_Leftarm: type revolute, parent Leftleg, child Leftarm, origin xyz=-1 0 0 rpy=0 0 0, axis 1 0 0, limit lower=-3.14159 upper=3.14159 effort=0.0 velocity=0.0
- added joint Rightleg_Rightarm: type revolute, parent Rightleg, child Rightarm, origin xyz=1 0 0 rpy=0 0 0, axis 1 0 0, limit lower=-3.14159 upper=3.14159 effort=0.0 velocity=0.0
- added joint Torso_Leftleg: type revolute, parent Torso, child Leftleg, origin xyz=-0.5 0 1 rpy=0 0 0, axis 1 0 0, limit lower=-3.14159 upper=3.14159 effort=0.0 velocity=0.0
- added joint Torso_Rightleg: type revolute, parent Torso, child Rightleg, origin xyz=0.5 0 1 rpy=0 0 0, axis 1 0 0, limit lower=-3.14159 upper=3.14159 effort=0.0 velocity=0.0
- joint Torso_Backleg: axis 0 1 0 -> 1 0 0; origin xyz=1 0 1 rpy=0 0 0 -> xyz=0 -0.5 1 rpy=0 0 0
- joint Torso_Frontleg: axis 0 1 0 -> 1 0 0; origin xyz=2 0 1 rpy=0 0 0 -> xyz=0 0.5 1 rpy=0 0 0
